File: MainBoard.sch (EAGLE design)
At the start: 66 parts, among them IC4 DS1307, IC7 74HC595D, IC8 74HC595D, IC9 74HC595D, U2 ATMEGA328P-AU

Commit message: - Added 3 Buttons - Organized Schematic
Parts:
- removed R27, R30, R31, R32: 47, rcl:R-EU_R0603
- added C11, C12, C13: 100nF, eagle-ltspice:CC0603
- added R11, R12, R13: 10k, eagle-ltspice:RR0603
- added R14, R15, R17, R18: 5R6, resistor:R-EU_R0805
- added S1, S2, S3: (no value), switch-omron:10-XX
- C3: value 47uF -> 100uF
- R10, R16, R5, R6, R7, R8, R9: value 47 -> 5R6; device rcl:R-EU_R0603 -> resistor:R-EU_R0805
- R2: value (none) -> r2
Connections:
- new net N$14: C12.1, R12.1, S2.S, U2.PD6
- new net N$15: C13.1, R13.1, S3.S, U2.PD7
- new net N$7: C11.1, R11.1, S1.S, U2.PD5
- net GND: now also C11.2, C12.2, C13.2, R11.2, R12.2, R13.2
- net N$1: now also R6.1; no longer R30.2
- net N$11: now also R14.1; no longer R5.2
- net N$2: now also R17.1; no longer R7.2
- net N$22: now also R10.1; no longer R9.2
- net N$23: now also R18.1; no longer R10.2
- net N$24: now also R15.1; no longer R16.2
- net N$3: now also R17.2; no longer R7.1
- net N$47: now also R6.2; no longer R30.1
- net N$50: now also R7.1; no longer R31.2
- net N$51: now also R7.2; no longer R31.1
- net N$52: now also R9.2; no longer R27.1
- net N$53: now also R16.1; no longer R8.2
- net N$54: now also R5.1; no longer R6.2
- net N$6: now also R9.1; no longer R27.2
- net N$71: now also R10.2; no longer R9.1
- net N$72: now also R8.2; no longer R32.1
- net N$74: now also R16.2; no longer R8.1
- net N$76: now also R18.2; no longer R10.1
- net N$77: now also R15.2; no longer R16.1
- net N$8: now also R8.1; no longer R32.2
- net N$80: now also R5.2; no longer R6.1
- net N$81: now also R14.2; no longer R5.1
- net VCC: now also S1.P, S2.P, S3.P
Other:
- moved on the sheet: JP1, JP10, JP11, JP12, JP13, JP14, JP15, JP16, JP17, JP18, JP19, JP2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

Commit message: Finished Routing an Panelizing
Parts:
- removed C3: 100uF, eagle-ltspice:CC0603
Connections:
- removed net +5V: C10.1, C7.2, U2.VCC, U2.VCC_2
- removed net N$4: C5.2, U2.AREF
- net GND: no longer C3.1
- net N$5: no longer C3.2
- net VCC: now also C10.1, C5.2, C7.2, U2.AREF, U2.VCC, U2.VCC_2
Other:
- moved on the sheet: C5, C7

Commit message: Changed tolerances on ledboard and mainboard
Parts:
- removed C13: 100nF, eagle-ltspice:CC0603
- removed IC9: 74HC595D, 74xx-eu:74HC595D
- removed JP1: (no value), pinhead:PINHD-2X2
- added C3: 100uF, eagle-ltspice:CC0603
- added IC1: DS1307, dallas:DS1307
- added JP31: (no value), pinhead:PINHD-2X3
- C1, C2: value 22uF -> 100uF
- C12: value 100nF -> 100uF
- C4, C5: value 100uF -> 22uF
- C8, C9: value 100uF -> 100nF
- IC4: value DS1307 -> 74HC595D; device dallas:DS1307 -> 74xx-eu:74HC595D
- JP12, JP13, JP16, JP18, JP3, JP6: device pinhead:PINHD-2X3 -> pinhead:PINHD-2X2
- JP22, JP23, JP26, JP27, JP29: device pinhead:PINHD-2X2 -> pinhead:PINHD-2X3
- R1, R11, R3, R4: value 10k -> 5R6; device eagle-ltspice:RR0603 -> resistor:R-EU_R0805
- R14, R18, R5, R6: value 5R6 -> 10k; device resistor:R-EU_R0805 -> eagle-ltspice:RR0603
- R2: value r2 -> 5R6; device eagle-ltspice:RR0603 -> resistor:R-EU_R0805
- R9: value 5R6 -> r2; device resistor:R-EU_R0805 -> eagle-ltspice:RR0603
- renumbered IC7 to IC2, IC8 to IC3, JP32 to PWR, U$2 to IC5, U$3 to IC6, U$4 to U$1, U2 to U1
Connections:
- net GND: now also C10.1, C12.1, C2.2, C3.1, C4.1, C6.2, C8.2, C9.2, IC1.GND, IC4A.G, JP22.3, JP23.3, JP26.3, JP27.3, JP29.3, JP31.3, R14.2, R18.2; no longer C10.2, C12.2, C13.2, C2.1, C4.2, C6.1, C8.1, C9.1, IC4.GND, IC9A.G, JP12.3, JP13.3, JP16.3, JP18.3, JP3.3, JP6.3, R11.2, R12.2
- net N$1: now also R11.1; no longer R6.1
- net N$11: now also R7.1; no longer R14.1
- net N$14: now also C9.1, R14.1; no longer C12.1, R12.1
- net N$15: now also C11.1, R18.1; no longer C13.1, R13.1
- net N$2: now also R16.1; no longer R17.1
- net N$22: now also R3.1; no longer R10.1
- net N$23: now also R2.1; no longer R18.1
- net N$24: now also R1.1; no longer R15.1
- net N$26: now also JP31.1; no longer JP3.1
- net N$27: now also IC1.VBAT; no longer IC4.VBAT
- net N$3: now also JP22.2, JP23.2, JP26.2, JP27.2, JP29.2, JP31.2, R16.2; no longer JP12.2, JP13.2, JP16.2, JP18.2, JP3.2, JP6.2, R17.2
- net N$32: now also IC1.SDA, R5.2; no longer IC4.SDA, R3.2
- net N$33: now also IC1.X2, R9.2; no longer IC4.X2, R2.2
- net N$37: now also IC1.X1, R9.1; no longer IC4.X1, R2.1
- net N$38: now also IC4A.QA, JP22.1; no longer IC9A.QA, JP12.1
- net N$39: now also IC1.SCL, R6.2; no longer IC4.SCL, R1.2
- net N$40: now also IC4A.QB, JP23.1; no longer IC9A.QB, JP13.1
- net N$44: now also C4.2; no longer C1.2
- net N$46: now also C5.2; no longer C2.2
- net N$47: now also JP12.1, JP13.1, JP15.1, JP16.1, JP18.1, JP19.1, JP21.1, R11.2; no longer JP11.1, JP2.1, JP23.1, JP26.1, JP29.1, JP5.1, JP8.1, R6.2
- net N$5: now also R12.1; no longer R4.1
- net N$50: now also R10.1; no longer R7.1
- net N$51: now also JP12.3, JP13.3, JP15.3, JP16.3, JP18.3, JP19.3, JP21.3, R10.2; no longer JP11.3, JP2.3, JP23.3, JP26.3, JP29.3, JP5.3, JP8.3, R7.2
- net N$52: now also JP22.5, JP23.5, JP26.5, JP27.5, JP29.5, JP31.5, R15.2; no longer JP12.5, JP13.5, JP16.5, JP18.5, JP3.5, JP6.5, R9.2
- net N$53: now also R4.1; no longer R16.1
- net N$54: now also R8.1; no longer R5.1
- net N$56: now also IC4A.QC, JP24.1; no longer IC9A.QC, JP16.1
- net N$57: now also IC4A.QD, JP25.1; no longer IC9A.QD, JP18.1
- net N$58: now also IC4A.QE, JP26.1; no longer IC9A.QE, JP24.1
- net N$6: now also R15.1; no longer R9.1
- net N$60: now also JP27.1; no longer JP28.1
- net N$62: now also JP28.1; no longer JP25.1
- net N$69: now also JP29.1; no longer JP30.1
- net N$7: now also C8.1, R13.1; no longer C11.1, R11.1
- net N$70: now also JP30.1; no longer JP6.1
- net N$71: now also JP11.1, JP2.1, JP3.1, JP5.1, JP6.1, JP8.1, R3.2; no longer JP1.1, JP15.1, JP19.1, JP21.1, JP22.1, JP27.1, R10.2
- net N$72: now also JP22.4, JP23.4, JP26.4, JP27.4, JP29.4, JP31.4, R17.2; no longer JP12.4, JP13.4, JP16.4, JP18.4, JP3.4, JP6.4, R8.2
- net N$74: now also JP11.3, JP2.3, JP3.3, JP5.3, JP6.3, JP8.3, R4.2; no longer JP1.3, JP15.3, JP19.3, JP21.3, JP22.3, JP27.3, R16.2
- net N$76: now also JP11.2, JP2.2, JP3.2, JP5.2, JP6.2, JP8.2, R2.2; no longer JP1.2, JP15.2, JP19.2, JP21.2, JP22.2, JP27.2, R18.2
- net N$77: now also JP11.4, JP2.4, JP3.4, JP5.4, JP6.4, JP8.4, R1.2; no longer JP1.4, JP15.4, JP19.4, JP21.4, JP22.4, JP27.4, R15.2
- net N$8: now also R17.1; no longer R8.1
- net N$80: now also JP12.2, JP13.2, JP15.2, JP16.2, JP18.2, JP19.2, JP21.2, R8.2; no longer JP11.2, JP2.2, JP23.2, JP26.2, JP29.2, JP5.2, JP8.2, R5.2
- net N$81: now also JP12.4, JP13.4, JP15.4, JP16.4, JP18.4, JP19.4, JP21.4, R7.2; no longer JP11.4, JP2.4, JP23.4, JP26.4, JP29.4, JP5.4, JP8.4, R14.2
- net N$9: now also IC4A.SER; no longer IC9A.SER
- net RCK: now also IC4A.RCK; no longer IC9A.RCK
- net SCK: now also IC4A.SCK; no longer IC9A.SCK
- net VCC: now also C1.2, C10.2, C12.2, C2.1, C3.2, C6.1, IC1.VCC, IC4A.SCL, JP22.6, JP23.6, JP26.6, JP27.6, JP29.6, JP31.6, R12.2, R5.1, R6.1; no longer C10.1, C4.1, C5.2, C6.2, C8.2, C9.2, IC4.VCC, IC9A.SCL, JP12.6, JP13.6, JP16.6, JP18.6, JP3.6, JP6.6, R1.1, R3.1, R4.2
Other:
- moved on the sheet: C1, C10, C11, C12, C2, C4, C5, C6, C7, C8, C9, JP10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

Commit message: Finalizing prototype
Parts:
- removed R9: r2, eagle-ltspice:RR0603
- added U$2: CC5V-T1A, cc5v-t1a:CC5V-T1A
Connections:
- removed net N$33: IC1.X2, R9.2
- removed net N$37: IC1.X1, R9.1
- new net N$16: IC1.X1, U$2.P$1
- new net N$4: IC1.X2, U$2.P$2
Changed lines of the file:
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@@
 <?xml version="1.0" encoding="utf-8"?>
 <!DOCTYPE eagle SYSTEM "eagle.dtd">
-<eagle version="6.4">
+<eagle version="6.5.0">
 <drawing>
 <settings>
@@
 <part name="GND19" library="supply1" deviceset="GND" device=""/>
 <part name="R6" library="eagle-ltspice" deviceset="R" device="R0603" value="10k"/>
-<part name="R9" library="eagle-ltspice" deviceset="R" device="R0603" value="r2"/>
 <part name="R5" library="eagle-ltspice" deviceset="R" device="R0603" value="10k"/>
 <part name="C1" library="eagle-ltspice" deviceset="C" device="C0603" value="100uF"/>
@@
 <part name="R2" library="resistor" deviceset="R-EU_" device="R0805" value="5R6"/>
 <part name="GND13" library="supply1" deviceset="GND" device=""/>
+<part name="U$2" library="cc5v-t1a" deviceset="CC5V-T1A" device=""/>
 </parts>
 <sheets>
@@
 <instance part="GND19" gate="1" x="48.26" y="137.16" rot="R180"/>
 <instance part="R6" gate="G$1" x="2.54" y="111.76"/>
-<instance part="R9" gate="G$1" x="40.64" y="104.14" rot="R90"/>
 <instance part="R5" gate="G$1" x="2.54" y="116.84"/>
 <instance part="C1" gate="G$1" x="-99.06" y="124.46"/>
@@
 <instance part="R2" gate="G$1" x="325.12" y="142.24"/>
 <instance part="GND13" gate="1" x="-106.68" y="116.84" rot="R180"/>
+<instance part="U$2" gate="G$1" x="40.64" y="104.14" rot="R180"/>
 </instances>
 <busses>
@@
 <pinref part="IC1" gate="G$1" pin="VBAT"/>
 <wire x1="48.26" y1="111.76" x2="33.02" y2="111.76" width="0.1524" layer="91"/>
-</segment>
-</net>
-<net name="N$33" class="0">
-<segment>
-<pinref part="IC1" gate="G$1" pin="X2"/>
-<wire x1="40.64" y1="109.22" x2="33.02" y2="109.22" width="0.1524" layer="91"/>
-<wire x1="33.02" y1="109.22" x2="33.02" y2="106.68" width="0.1524" layer="91"/>
-<pinref part="R9" gate="G$1" pin="2"/>
-</segment>
-</net>
-<net name="N$37" class="0">
-<segment>
-<pinref part="IC1" gate="G$1" pin="X1"/>
-<wire x1="40.64" y1="99.06" x2="33.02" y2="99.06" width="0.1524" layer="91"/>
-<wire x1="33.02" y1="99.06" x2="33.02" y2="101.6" width="0.1524" layer="91"/>
-<pinref part="R9" gate="G$1" pin="1"/>
 </segment>
 </net>
@@
 </segment>
 </net>
+<net name="N$4" class="0">
+<segment>
+<pinref part="IC1" gate="G$1" pin="X2"/>
+<pinref part="U$2" gate="G$1" pin="P$2"/>
+<wire x1="33.02" y1="106.68" x2="35.56" y2="106.68" width="0.1524" layer="91"/>
+</segment>
+</net>
+<net name="N$16" class="0">
+<segment>
+<pinref part="U$2" gate="G$1" pin="P$1"/>
+<pinref part="IC1" gate="G$1" pin="X1"/>
+<wire x1="35.56" y1="101.6" x2="33.02" y2="101.6" width="0.1524" layer="91"/>
+</segment>
+</net>
 </nets>
 </sheet>
 </sheets>
-<errors>
-</errors>
 </schematic>
 </drawing>

Commit message: Final layout of prototype
Parts:
- removed Q1: (no value), crystal:CRYSTALCTS406
- added U$3: 16,00-MT, 1600MT:16,00-MT
- C4, C5: value 22uF -> (none); device eagle-ltspice:CC0603 -> rcl:C-EUC0603
Connections:
- removed net N$46: C5.2, Q1.1, U1.PB7
- new net N$17: C5.2, U$3.P$2, U1.PB7
- net N$44: now also U$3.P$1; no longer Q1.2
Changed lines of the file:
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@@
 <?xml version="1.0" encoding="utf-8"?>
 <!DOCTYPE eagle SYSTEM "eagle.dtd">
-<eagle version="6.5.0">
+<eagle version="6.4">
 <drawing>
 <settings>
@@
 <part name="C1" library="eagle-ltspice" deviceset="C" device="C0603" value="100uF"/>
 <part name="C3" library="eagle-ltspice" deviceset="C" device="C0603" value="100uF"/>
-<part name="C4" library="eagle-ltspice" deviceset="C" device="C0603" value="22uF"/>
-<part name="C5" library="eagle-ltspice" deviceset="C" device="C0603" value="22uF"/>
 <part name="R12" library="eagle-ltspice" deviceset="R" device="R0603" value="10k"/>
 <part name="C6" library="eagle-ltspice" deviceset="C" device="C0603" value="100uF"/>
@@
 <part name="JP19" library="pinhead" deviceset="PINHD-2X2" device=""/>
 <part name="JP29" library="pinhead" deviceset="PINHD-2X3" device=""/>
-<part name="Q1" library="crystal" deviceset="CRYSTAL" device="CTS406"/>
 <part name="PWR" library="pinhead" deviceset="PINHD-2X2" device=""/>
 <part name="JP2" library="pinhead" deviceset="PINHD-2X2" device=""/>
@@
 <part name="GND13" library="supply1" deviceset="GND" device=""/>
 <part name="U$2" library="cc5v-t1a" deviceset="CC5V-T1A" device=""/>
+<part name="U$3" library="1600MT" deviceset="16,00-MT" device=""/>
+<part name="C4" library="rcl" deviceset="C-EU" device="C0603"/>
+<part name="C5" library="rcl" deviceset="C-EU" device="C0603"/>
 </parts>
 <sheets>
@@
 <instance part="C1" gate="G$1" x="-99.06" y="124.46"/>
 <instance part="C3" gate="G$1" x="-106.68" y="109.22"/>
-<instance part="C4" gate="G$1" x="-121.92" y="86.36" rot="R90"/>
-<instance part="C5" gate="G$1" x="-129.54" y="81.28" rot="R90"/>
 <instance part="R12" gate="G$1" x="-30.48" y="78.74" rot="R90"/>
 <instance part="C6" gate="G$1" x="-30.48" y="58.42" rot="R180"/>
@@
 <instance part="JP19" gate="A" x="454.66" y="101.6" rot="R90"/>
 <instance part="JP29" gate="A" x="208.28" y="-162.56"/>
-<instance part="Q1" gate="G$1" x="-114.3" y="83.82" rot="R90"/>
 <instance part="PWR" gate="A" x="-15.24" y="154.94"/>
 <instance part="JP2" gate="A" x="345.44" y="134.62" rot="R90"/>
@@
 <instance part="GND13" gate="1" x="-106.68" y="116.84" rot="R180"/>
 <instance part="U$2" gate="G$1" x="40.64" y="104.14" rot="R180"/>
+<instance part="U$3" gate="G$1" x="-114.3" y="83.82"/>
+<instance part="C4" gate="G$1" x="-121.92" y="86.36" rot="R90"/>
+<instance part="C5" gate="G$1" x="-129.54" y="81.28" rot="R90"/>
 </instances>
 <busses>
@@
 <net name="N$44" class="0">
 <segment>
-<wire x1="-109.22" y1="86.36" x2="-114.3" y2="86.36" width="0.1524" layer="91"/>
-<wire x1="-114.3" y1="86.36" x2="-116.84" y2="86.36" width="0.1524" layer="91"/>
-<wire x1="-109.22" y1="83.82" x2="-109.22" y2="86.36" width="0.1524" layer="91"/>
 <wire x1="-81.28" y1="83.82" x2="-109.22" y2="83.82" width="0.1524" layer="91"/>
 <pinref part="U1" gate="A" pin="PB6"/>
+<wire x1="-109.22" y1="83.82" x2="-109.22" y2="86.36" width="0.1524" layer="91"/>
+<wire x1="-109.22" y1="86.36" x2="-114.3" y2="86.36" width="0.1524" layer="91"/>
+<pinref part="U$3" gate="G$1" pin="P$1"/>
+<wire x1="-114.3" y1="86.36" x2="-116.84" y2="86.36" width="0.1524" layer="91"/>
+<junction x="-114.3" y="86.36"/>
 <pinref part="C4" gate="G$1" pin="2"/>
-<pinref part="Q1" gate="G$1" pin="2"/>
-<junction x="-114.3" y="86.36"/>
-</segment>
-</net>
-<net name="N$46" class="0">
-<segment>
-<wire x1="-81.28" y1="81.28" x2="-114.3" y2="81.28" width="0.1524" layer="91"/>
-<pinref part="U1" gate="A" pin="PB7"/>
-<pinref part="C5" gate="G$1" pin="2"/>
-<pinref part="Q1" gate="G$1" pin="1"/>
-<wire x1="-114.3" y1="81.28" x2="-124.46" y2="81.28" width="0.1524" layer="91"/>
-<junction x="-114.3" y="81.28"/>
 </segment>
 </net>
@@
 </segment>
 </net>
+<net name="N$17" class="0">
+<segment>
+<pinref part="U1" gate="A" pin="PB7"/>
+<wire x1="-81.28" y1="81.28" x2="-114.3" y2="81.28" width="0.1524" layer="91"/>
+<pinref part="U$3" gate="G$1" pin="P$2"/>
+<wire x1="-114.3" y1="81.28" x2="-124.46" y2="81.28" width="0.1524" layer="91"/>
+<pinref part="C5" gate="G$1" pin="2"/>
+</segment>
+</net>
